File: hardware/LED Driver STM/LED Driver STM.sch (KiCad schematic (older format))
At the start: 39 parts

Commit message: Updated layout
Parts:
- J1: renamed from J?; footprint (none) -> Connector_PinHeader_2.54mm:PinHeader_1x04_P2.54mm_Vertical
- SW1, SW2, SW3: renamed from SW?; footprint (none) -> LCSC:SW_TS-1187A-B-A-B; symbol Switch:SW_Push -> LCSC_Button:TS-1187A-B-A-B
- gave numbers to parts that had none: 35
Connections:
- net BOOT0: now also SW2.C, SW2.D; no longer SW2.2
- net CS1: no longer U3.5 (CS)
- net CS2: now also U3.5 (CS)
- net GND: now also SW1.A, SW1.B, SW2.A, SW2.B, SW3.A, SW3.B; no longer SW1.1, SW2.1, SW3.1
- net NRST: now also SW1.C, SW1.D; no longer SW1.2
- net SW1: now also SW3.C, SW3.D; no longer SW3.2
