File: hardware/LED-Driver-STM/LED-Driver-STM.sch (KiCad schematic (older format))
At the start: 39 parts, among them J1 I2C4, J2 IO5, J3 PWR, J4 PROG5, J5 ADC2, J6 INT2, J7 INT2, J8 ADC3, SW1 SPT, SW2 SPT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

Commit message: Finished Routing V1
Parts:
- added C14: 10u_25v, Capacitor_SMD:C_0805_2012Metric, symbol Device:C_Small
- added C15, C16, C17: 100n, Capacitor_SMD:C_0402_1005Metric, symbol Device:C_Small
- C1, C4: LCSC (none) -> C1547
- C10, C12: LCSC (none) -> C15525
- C11, C13, C9: LCSC (none) -> C1525
- C2, C3, C5, C8: LCSC (none) -> C15195
- C6: LCSC (none) -> C52923
- C7: LCSC (none) -> C15850
- D1: LCSC (none) -> C8598
- D2: LCSC (none) -> C2286
- L1: LCSC (none) -> C26443
- R1, R2, R6: LCSC (none) -> C11702
- R3: LCSC (none) -> C25118
- R4, R5: LCSC (none) -> C25744
- R7: LCSC (none) -> C25133
- SW1, SW2, SW3: symbol LCSC_Button:TS-1187A-B-A-B -> LED-Driver-STM-rescue:TS-1187A-B-A-B-LCSC_Button-LED-Driver-STM-rescue; LCSC (none) -> C318884
- U1: LCSC (none) -> C23922
- U2: LCSC (none) -> C6186
- U3: LCSC (none) -> C26444
- U4: LCSC (none) -> C15134
- Y1: LCSC (none) -> C13738
Connections:
- wire segments 204 -> 222
Other:
- moved on the sheet: C12, C13, C6, C8, L1

Commit message: Latest board layout
This is the board that was purchased
Parts:
- SW1, SW2, SW3: symbol LED-Driver-STM-rescue:TS-1187A-B-A-B-LCSC_Button-LED-Driver-STM-rescue -> LED-Driver-STM-rescue:TS-1187A-B-A-B-LCSC_Button-LED-Driver-STM-rescue-LED-Driver-STM-rescue
Changed lines of the file:
@@
 $EndComp
 $Comp
-L LED-Driver-STM-rescue:TS-1187A-B-A-B-LCSC_Button-LED-Driver-STM-rescue SW1
+L LED-Driver-STM-rescue:TS-1187A-B-A-B-LCSC_Button-LED-Driver-STM-rescue-LED-Driver-STM-rescue SW1
 U 1 1 5F7153FD
 P 700 1900
@@
 $EndComp
 $Comp
-L LED-Driver-STM-rescue:TS-1187A-B-A-B-LCSC_Button-LED-Driver-STM-rescue SW2
+L LED-Driver-STM-rescue:TS-1187A-B-A-B-LCSC_Button-LED-Driver-STM-rescue-LED-Driver-STM-rescue SW2
 U 1 1 5F71DB9F
 P 700 2850
@@
 $EndComp
 $Comp
-L LED-Driver-STM-rescue:TS-1187A-B-A-B-LCSC_Button-LED-Driver-STM-rescue SW3
+L LED-Driver-STM-rescue:TS-1187A-B-A-B-LCSC_Button-LED-Driver-STM-rescue-LED-Driver-STM-rescue SW3
 U 1 1 5F86A090
 P 1650 2850
